File: GPSHolder.sch (KiCad schematic (older format))
At the start: 7 parts, among them J1 TEST_1P, J2 TEST_1P, J3 TEST_1P, J4 TEST_1P

Commit message: Add files via upload
Parts:
- removed L_Conn1, R_Conn1: Conn_01x06_Male, Pin_Headers:Pin_Header_Angled_1x06_Pitch2.54mm, symbol Conn_01x06_Male
- added L_Conn1, R_Conn1: Conn_01x08_Male, Pin_Headers:Pin_Header_Angled_1x08_Pitch2.54mm, symbol Conn_01x08_Male
Connections:
- net at Molex1.4 (Pin_4): now also L_Conn1.3 (Pin_3)
- net at Molex1.3 (Pin_3): now also L_Conn1.4 (Pin_4)
- net at Molex1.1 (Pin_1): now also R_Conn1.2 (Pin_2)
- net at Molex1.2 (Pin_2): now also R_Conn1.1 (Pin_1)
Changed lines of the file:
@@
 $EndDescr
-$Comp
-L Conn_01x06_Male L_Conn1
-U 1 1 5AEC9C40
-P 4900 3800
-F 0 "L_Conn1" H 4900 4100 50  0000 C CNN
-F 1 "Conn_01x06_Male" H 4900 3400 50  0000 C CNN
-F 2 "Pin_Headers:Pin_Header_Angled_1x06_Pitch2.54mm" H 4900 3800 50  0001 C CNN
-F 3 "" H 4900 3800 50  0001 C CNN
-	1    4900 3800
-	1    0    0    -1
-$EndComp
-$Comp
-L Conn_01x06_Male R_Conn1
-U 1 1 5AEC9D4C
-P 4900 4725
-F 0 "R_Conn1" H 4900 5025 50  0000 C CNN
-F 1 "Conn_01x06_Male" H 4900 4325 50  0000 C CNN
-F 2 "Pin_Headers:Pin_Header_Angled_1x06_Pitch2.54mm" H 4900 4725 50  0001 C CNN
-F 3 "" H 4900 4725 50  0001 C CNN
-	1    4900 4725
-	1    0    0    -1
-$EndComp
 $Comp
 L Conn_01x04_Male Molex1
@@
 	-1   0    0    1
 $EndComp
-Wire Wire Line
-	5950 4175 5950 3600
-Wire Wire Line
-	5950 3600 5100 3600
-Wire Wire Line
-	5950 4275 5850 4275
-Wire Wire Line
-	5850 4275 5850 3700
-Wire Wire Line
-	5850 3700 5100 3700
-Wire Wire Line
-	5950 4375 5825 4375
-Wire Wire Line
-	5825 4375 5825 5025
-Wire Wire Line
-	5825 5025 5100 5025
-Wire Wire Line
-	5950 4475 5950 4925
-Wire Wire Line
-	5950 4925 5100 4925
-Text Label 4750 4925 0    39   ~ 0
-3.3V
-Text Label 4750 5025 0    39   ~ 0
-GND
 Text Label 4775 3600 0    39   ~ 0
 TXD
@@
 	1    0    0    -1
 $EndComp
+$Comp
+L Conn_01x08_Male L_Conn1
+U 1 1 5AEE312A
+P 4900 3700
+F 0 "L_Conn1" H 4900 4100 50  0000 C CNN
+F 1 "Conn_01x08_Male" H 4900 3200 50  0000 C CNN
+F 2 "Pin_Headers:Pin_Header_Angled_1x08_Pitch2.54mm" H 4900 3700 50  0001 C CNN
+F 3 "" H 4900 3700 50  0001 C CNN
+	1    4900 3700
+	1    0    0    -1
+$EndComp
+$Comp
+L Conn_01x08_Male R_Conn1
+U 1 1 5AEE31A5
+P 4900 4675
+F 0 "R_Conn1" H 4900 5075 50  0000 C CNN
+F 1 "Conn_01x08_Male" H 4900 4175 50  0000 C CNN
+F 2 "Pin_Headers:Pin_Header_Angled_1x08_Pitch2.54mm" H 4900 4675 50  0001 C CNN
+F 3 "" H 4900 4675 50  0001 C CNN
+	1    4900 4675
+	1    0    0    -1
+$EndComp
+Text Label 4750 5000 0    39   ~ 0
+3.3V
+Text Label 4750 5100 0    39   ~ 0
+GND
+Wire Wire Line
+	5950 4175 5950 3600
+Wire Wire Line
+	5950 3600 5100 3600
+Wire Wire Line
+	5950 4275 5850 4275
+Wire Wire Line
+	5850 4275 5850 3700
+Wire Wire Line
+	5850 3700 5100 3700
 Wire Wire Line
 	6750 4200 6750 4350
@@
 	7250 4450 7250 4350
 Connection ~ 7250 4350
+Wire Wire Line
+	5950 4375 5100 4375
+Wire Wire Line
+	5950 4475 5100 4475
 $EndSCHEMATC

Commit message: Final design. Schematic pdf and gerbers generated
Parts:
- Molex1: footprint SOAR_Library:Molex_Micro-Fit_3.0_43045-0400_2x02_P3.00mm_Horizontal -> SOAR_Kicad_Library:Molex_Micro-Fit_3.0_43045-0400_2x02_P3.00mm_Horizontal
Connections:
- net GND: now also L_Conn1.8 (Pin_8), Molex1.2 (Pin_2), R_Conn1.8 (Pin_8)
- net at Molex1.1 (Pin_1): now also R_Conn1.7 (Pin_7); no longer R_Conn1.2 (Pin_2)
- net at R_Conn1.1 (Pin_1): no longer Molex1.2 (Pin_2)
Changed lines of the file:
@@
 F 0 "Molex1" H 6150 4075 50  0000 C CNN
 F 1 "Conn_01x04_Male" H 6025 4575 50  0000 C CNN
-F 2 "SOAR_Library:Molex_Micro-Fit_3.0_43045-0400_2x02_P3.00mm_Horizontal" H 6150 4375 50  0001 C CNN
+F 2 "SOAR_Kicad_Library:Molex_Micro-Fit_3.0_43045-0400_2x02_P3.00mm_Horizontal" H 6150 4375 50  0001 C CNN
 F 3 "" H 6150 4375 50  0001 C CNN
 	1    6150 4375
@@
 Connection ~ 7250 4350
 Wire Wire Line
-	5950 4375 5100 4375
+	5785 4375 5950 4375
 Wire Wire Line
-	5950 4475 5100 4475
+	5785 4375 5785 4725
+Wire Wire Line
+	5785 4725 5975 4725
+Wire Wire Line
+	5975 4725 5975 5075
+Wire Wire Line
+	5975 5075 5100 5075
+Wire Wire Line
+	5100 4975 5570 4975
+Wire Wire Line
+	5570 4975 5570 4475
+Wire Wire Line
+	5570 4475 5950 4475
+$Comp
+L GND #PWR02
+U 1 1 5AFAAB2B
+P 5590 5115
+F 0 "#PWR02" H 5590 4865 50  0001 C CNN
+F 1 "GND" H 5590 4965 50  0000 C CNN
+F 2 "" H 5590 5115 50  0001 C CNN
+F 3 "" H 5590 5115 50  0001 C CNN
+	1    5590 5115
+	1    0    0    -1
+$EndComp
+Wire Wire Line
+	5590 5075 5590 5115
+Connection ~ 5590 5075
+$Comp
+L GND #PWR03
+U 1 1 5AFAAC30
+P 5340 4125
+F 0 "#PWR03" H 5340 3875 50  0001 C CNN
+F 1 "GND" H 5340 3975 50  0000 C CNN
+F 2 "" H 5340 4125 50  0001 C CNN
+F 3 "" H 5340 4125 50  0001 C CNN
+	1    5340 4125
+	1    0    0    -1
+$EndComp
+Wire Wire Line
+	5100 4100 5340 4100
+Wire Wire Line
+	5340 4100 5340 4125
 $EndSCHEMATC
